File: hardware/sensors/bmp581/BMP_unit.kicad_sch (KiCad schematic)
At the start: 4 parts, among them U1 BMP581

Commit message: Redo Schematic Upload
Reupload to test uploading from Github Desktop
Parts:
- removed D1: D, Diode_THT:D_DO-35_SOD27_P7.62mm_Horizontal, symbol Device:D
- removed R1: 100kohm, Package_DIP:DIP-8_W7.62mm, symbol Device:R_US
Connections:
- net MISO_out is gone; now on net GND: U1.5 (SDO)
- net +3.3V: now also U1.6 (CSB)
- net GND: no longer U1.7 (INT)
- net MOSI_out renamed SDI_3V
- net SerialCLK renamed SCK_3V
Other:
- moved on the sheet: C1
